File: PCB/TxTroller.kicad_sch (KiCad schematic)
At the start: 7 parts, among them J1 RadioReceiver, Q1 2N2222, U1 XIAO-RP2040-DIP

Commit message: fixed pin assignments
Connections:
- net SBUS_STAT: now also U1.7 (GPIO0/TX); no longer U1.8 (GPIO1/RX)
- net at Q1.3 (C), R_INV1.2: now also U1.8 (GPIO1/RX); no longer U1.7 (GPIO0/TX)
Changed lines of the file:
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@@
+	(wire
+		(pts
+			(xy 27.94 67.31) (xy 40.64 67.31)
+		)
+		(stroke
+			(width 0)
+			(type default)
+		)
+	)
 	(wire
 		(pts
@@
 	(wire
 		(pts
-			(xy 31.75 67.31) (xy 40.64 67.31)
-		)
-		(stroke
-			(width 0)
-			(type default)
-		)
-	)
-	(wire
-		(pts
 			(xy 154.94 54.61) (xy 154.94 57.15)
 		)
@@
 	)
 	(label "GPIO_0"
-		(at 31.75 67.31 0)
+		(at 88.9 67.31 180)
 		(effects
 			(font
 				(size 1.27 1.27)
 			)
-			(justify left bottom)
+			(justify right bottom)
 		)
 	)
@@
 	)
 	(label "SBUS_STAT"
-		(at 88.9 67.31 180)
+		(at 27.94 67.31 0)
 		(effects
 			(font
 				(size 1.27 1.27)
 			)
-			(justify right bottom)
-		)
-	)
+			(justify left bottom)
+		)
+	)
